Commit message: Fix lidar_joint origin height in URDF file (15cm)

File: src/scout_mini_ros2/scout_sim/urdf/scout_mini.urdf.xacro (robot description, xacro)
@@ -145,5 +145,5 @@
     <parent link="base_link"/>
     <child  link="lidar_link"/>
-    <origin xyz="0.0 0.0 ${base_height/2 + lidar_height}" rpy="0 0 0"/>
+    <origin xyz="0.0 0.0 0.15" rpy="0 0 0"/>
   </joint>
   <!-- ═══════════════════ IMU ══════════════════════════════════════════ -->

Commit message: pi warning is fixed.
redefining global symbol: pi

File: src/scout_mini_ros2/scout_sim/urdf/scout_mini.urdf.xacro (robot description, xacro)
@@ -36,5 +36,4 @@
   <xacro:property name="wheelbase"     value="0.498"/>  <!-- front-to-rear axle distance -->
   <xacro:property name="lidar_height"  value="0.25"/>   <!-- above base_link origin -->
-  <xacro:property name="pi"            value="3.14159265358979"/>
   <!-- ═══════════════════ MACROS ═══════════════════════════════════════ -->
   <xacro:macro name="box_inertia" params="m l w h">

Commit message: nav2 configurations, nav launch file

File: src/scout_mini_ros2/scout_sim/urdf/scout_mini.urdf.xacro (robot description, xacro)
@@ -24,5 +24,9 @@
 <robot name="scout_mini" xmlns:xacro="http://www.ros.org/wiki/xacro">
   <!-- ═══════════════════ PARAMETERS ═══════════════════════════════════ -->
-  <xacro:property name="mesh_path" value="$(find scout_sim)/meshes"/>
+  <!-- Mesh paths use the ROS 2 "package://" URI scheme so they resolve
+       cleanly in RViz (Ogre) AND Gazebo regardless of OS / mount type.
+       Absolute paths via $(find scout_sim) work in Gazebo but RViz on
+       WSL2 sometimes fails to read /mnt/c/... paths reliably. -->
+  <xacro:property name="mesh_path" value="package://scout_sim/meshes"/>
   <xacro:property name="base_length"   value="0.600"/>  <!-- m -->
   <xacro:property name="base_width"    value="0.450"/>  <!-- m -->
@@ -183,9 +187,15 @@
       <wheel_separation>${track_width}</wheel_separation>
       <wheel_radius>${wheel_radius}</wheel_radius>
-      <!-- ROS2 topic names — leading slash = publish to global Gazebo topic,
-           matching what ros_gz_bridge bridges from /tf → ROS /tf -->
+      <!-- ROS2 topic for velocity commands -->
       <topic>/cmd_vel</topic>
-      <odom_topic>/odom</odom_topic>
-      <tf_topic>/tf</tf_topic>
+      <!-- DiffDrive's odom output is DISABLED.  The wheel-encoder
+           integration is unreliable for skid-steer (wheels slip during
+           rotation, so encoders report rotation that didn't physically
+           happen).  We use the OdometryPublisher plugin below to publish
+           ground-truth odometry from Gazebo's physics state instead.
+           These topic names are intentionally non-bridged so the bridge
+           never sees them. -->
+      <odom_topic>/diff_drive_odom_unused</odom_topic>
+      <tf_topic>/diff_drive_tf_unused</tf_topic>
       <frame_id>odom</frame_id>
       <child_frame_id>base_footprint</child_frame_id>
@@ -193,4 +203,47 @@
       <max_linear_acceleration>1.0</max_linear_acceleration>
       <max_angular_acceleration>2.0</max_angular_acceleration>
+    </plugin>
+  </gazebo>
+  <!-- ═══════════════════ ODOMETRY PUBLISHER (ground truth) ═══════════ -->
+  <!--
+    Publishes the chassis's TRUE pose from Gazebo's physics state, not
+    from wheel encoders.  This solves the skid-steer slip problem: when
+    wheels spin in place, ground-truth says "no motion" so odom and TF
+    stay still, and the lidar doesn't appear to rotate in the map.
+    Educationally: this is "cheating" — real robots can't see their
+    own pose this way.  Real-world solutions involve IMU + wheel-encoder
+    fusion (e.g. robot_localization's EKF).  For this teaching exercise,
+    we trade a tiny bit of realism for a major reduction in confusion.
+  -->
+  <gazebo>
+    <plugin filename="gz-sim-odometry-publisher-system"
+            name="gz::sim::systems::OdometryPublisher">
+      <odom_frame>odom</odom_frame>
+      <robot_base_frame>base_footprint</robot_base_frame>
+      <odom_publish_frequency>50</odom_publish_frequency>
+      <odom_topic>/odom</odom_topic>
+      <tf_topic>/tf</tf_topic>
+      <dimensions>2</dimensions>
+    </plugin>
+  </gazebo>
+  <!-- ═══════════════════ VELOCITY CONTROL (chassis motion) ═══════════ -->
+  <!--
+    Directly enforces the chassis's linear and angular velocity from
+    /cmd_vel, bypassing wheel-ground physics entirely.  This solves the
+    skid-steer rotation problem: when MPPI commands "rotate at 0.5 rad/s"
+    the chassis ACTUALLY rotates at 0.5 rad/s — no slip, no friction
+    artifacts, no "Failed to make progress" timeouts.
+    DiffDrive (above) still subscribes to /cmd_vel and spins the wheel
+    joints, so wheels visually rotate. But the chassis pose is dictated
+    by VelocityControl, not by wheel-ground friction.
+    Educationally: this is "kinematic" simulation rather than "dynamic" —
+    common practice in Nav2 teaching demos so students learn navigation
+    concepts without debugging Gazebo's notoriously finicky skid-steer
+    friction. Real hardware tests still validate true wheel physics.
+  -->
+  <gazebo>
+    <plugin filename="gz-sim-velocity-control-system"
+            name="gz::sim::systems::VelocityControl">
+      <topic>/cmd_vel</topic>
     </plugin>
   </gazebo>

Commit message: Fix scout_mini.urdf.xacro

File: src/scout_mini_ros2/scout_sim/urdf/scout_mini.urdf.xacro (robot description, xacro)
@@ -24,9 +24,11 @@
 <robot name="scout_mini" xmlns:xacro="http://www.ros.org/wiki/xacro">
   <!-- ═══════════════════ PARAMETERS ═══════════════════════════════════ -->
-  <!-- Mesh paths use the ROS 2 "package://" URI scheme so they resolve
-       cleanly in RViz (Ogre) AND Gazebo regardless of OS / mount type.
-       Absolute paths via $(find scout_sim) work in Gazebo but RViz on
-       WSL2 sometimes fails to read /mnt/c/... paths reliably. -->
-  <xacro:property name="mesh_path" value="package://scout_sim/meshes"/>
+  <!-- Mesh paths use the ROS 2 "package://" URI scheme:
+         - RViz: resolves via ROS package paths.
+         - Gazebo: ros_gz_sim translates package:// → model://, which
+           then resolves because we registered scout_sim as a model
+           via the model.config file at the package root.
+       Together this works for both engines without absolute paths. -->
+  <xacro:property name="mesh_path" value="$(find scout_sim)/meshes"/>
   <xacro:property name="base_length"   value="0.600"/>  <!-- m -->
   <xacro:property name="base_width"    value="0.450"/>  <!-- m -->

Commit message: Fix some bugs

File: src/scout_mini_ros2/scout_sim/urdf/scout_mini.urdf.xacro (robot description, xacro)
@@ -30,5 +30,5 @@
            via the model.config file at the package root.
        Together this works for both engines without absolute paths. -->
-  <xacro:property name="mesh_path" value="$(find scout_sim)/meshes"/>
+  <xacro:property name="mesh_path" value="package://scout_sim/meshes"/>
   <xacro:property name="base_length"   value="0.600"/>  <!-- m -->
   <xacro:property name="base_width"    value="0.450"/>  <!-- m -->
@@ -259,5 +259,5 @@
       <always_on>true</always_on>
       <visualize>true</visualize>
-      <topic>scan</topic>
+      <topic>/scout_mini/scan</topic>
       <gz_frame_id>lidar_link</gz_frame_id>
       <lidar>
@@ -296,5 +296,5 @@
       <update_rate>100</update_rate>
       <always_on>true</always_on>
-      <topic>imu/data</topic>
+      <topic>/scout_mini/imu/data</topic>
       <imu>
         <angular_velocity>
